File: imx219_mipi24/imx219_mipi24.kicad_pcb (KiCad board)
At the start: 4 copper layers, 25 x 25 mm, 33 parts, among them J1 DF37NC-30DS-0.4V(51), J2 FH52-24S-0.5SH, U1 RT9193-18GB, U2 AP7331-28WG, U3 LM3671MF-1.2/NOPB, X1 SG-8101CG 24.000000MHz

Commit message: update
Other:
- board text added: "RTCL-IMX219-MIPI24-V2"
- board text removed: "RCL-IMX219-MIPI24-V1"
Changed lines of the file:
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@@
 		(at 148.5 92.5 180)
 		(property "Reference" "J1"
-			(at 5.1 -0.05 180)
+			(at 5.2 -0.1 270)
 			(layer "F.SilkS")
 			(effects
@@
 		(layer "User.1")
 	)
-	(gr_text "RCL-IMX219-MIPI24-V1"
-		(at 140.5 89.5 0)
+	(gr_text "RTCL-IMX219-MIPI24-V2\n"
+		(at 160.3 109.8 180)
 		(layer "F.SilkS")
 		(effects
